File: 555Trigger/_autosave-555Trigger.kicad_sch (KiCad schematic)
At the start: 11 parts, among them J1 Conn_01x03_Socket, J2 Timing Signal Out, J3 Timing Signal In, U1 L272, U2 TLC555xP

Commit message: added filtering and buffers to circuit todo: make one large master control board
Parts:
- C3: value C -> 2.2 μF
- J1: value Conn_01x03_Socket -> Power Signal Input
- R2: value R -> 10K
- renumbered U2 to 555Timer
Other:
- moved on the sheet: R2
Changed lines of the file:
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@@
     (stroke (width 0) (type default))
   )
-  (wire (pts (xy 87.63 85.09) (xy 96.52 85.09))
+  (wire (pts (xy 90.17 85.09) (xy 96.52 85.09))
     (stroke (width 0) (type default))
   )
@@
   )
   (wire (pts (xy 170.18 95.25) (xy 161.29 95.25))
+    (stroke (width 0) (type default))
+  )
+  (wire (pts (xy 82.55 85.09) (xy 80.01 85.09))
     (stroke (width 0) (type default))
   )
@@
       (effects (font (size 1.27 1.27)))
     )
-    (property "Value" "Conn_01x03_Socket" (at 75.565 82.55 0)
+    (property "Value" "Power Signal Input" (at 75.565 82.55 0)
       (effects (font (size 1.27 1.27)))
     )
@@
   (symbol (lib_id "Timer:TLC555xP") (at 148.59 90.17 0) (unit 1)
     (in_bom yes) (on_board yes) (dnp no) (fields_autoplaced)
-    (property "Reference" "U2" (at 150.7841 77.47 0)
+    (property "Reference" "555Timer" (at 150.7841 77.47 0)
       (effects (font (size 1.27 1.27)) (justify left))
     )
@@
       (project "555Trigger"
         (path "/ddfde45b-0759-482c-9a42-ae9b2feffe30"
-          (reference "U2") (unit 1)
+          (reference "555Timer") (unit 1)
         )
       )
@@
   (symbol (lib_id "Device:C") (at 170.18 100.33 0) (unit 1)
     (in_bom yes) (on_board yes) (dnp no)
-    (property "Reference" "C1" (at 182.88 101.6 0)
-      (effects (font (size 1.27 1.27)) (justify left))
-    )
-    (property "Value" "2.2 μF" (at 182.88 104.14 0)
+    (property "Reference" "C1" (at 175.26 100.33 0)
+      (effects (font (size 1.27 1.27)) (justify left))
+    )
+    (property "Value" "2.2 μF" (at 175.26 104.14 0)
       (effects (font (size 1.27 1.27)) (justify left))
     )
@@
       (effects (font (size 1.27 1.27)) (justify left))
     )
-    (property "Value" "C" (at 100.33 95.25 0)
+    (property "Value" "2.2 μF" (at 100.33 95.25 0)
       (effects (font (size 1.27 1.27)) (justify left))
     )
@@
     )
   )
-  (symbol (lib_id "Device:R") (at 83.82 85.09 90) (unit 1)
-    (in_bom yes) (on_board yes) (dnp no) (fields_autoplaced)
-    (property "Reference" "R2" (at 83.82 78.74 90)
-      (effects (font (size 1.27 1.27)))
-    )
-    (property "Value" "R" (at 83.82 81.28 90)
-      (effects (font (size 1.27 1.27)))
-    )
-    (property "Footprint" "Resistor_THT:R_Axial_DIN0204_L3.6mm_D1.6mm_P5.08mm_Horizontal" (at 83.82 86.868 90)
-      (effects (font (size 1.27 1.27)) hide)
-    )
-    (property "Datasheet" "~" (at 83.82 85.09 0)
-      (effects (font (size 1.27 1.27)) hide)
-    )
+  (symbol (lib_id "Device:R") (at 86.36 85.09 90) (unit 1)
+    (in_bom yes) (on_board yes) (dnp no) (fields_autoplaced)
+    (property "Reference" "R2" (at 86.36 78.74 90)
+      (effects (font (size 1.27 1.27)))
+    )
+    (property "Value" "10K" (at 86.36 81.28 90)
+      (effects (font (size 1.27 1.27)))
+    )
+    (property "Footprint" "Resistor_THT:R_Axial_DIN0204_L3.6mm_D1.6mm_P5.08mm_Horizontal" (at 86.36 86.868 90)
+      (effects (font (size 1.27 1.27)) hide)
+    )
+    (property "Datasheet" "~" (at 86.36 85.09 0)
+      (effects (font (size 1.27 1.27)) hide)
+    )
